File: kicad/ir_to_usb/ir_to_usb.sch (KiCad schematic (older format))
At the start: 12 parts, among them J1 Conn_01x04_Male, Q1 BC337, U1 ArduinoProMicro

Commit message: Update schematics.
Connections:
- net GND: now also R2.1, R3.1
- net at R3.2, U1.~ (Vin): now also J1.3 (Pin_3)
- net at R2.2, U1.~ (Vin): now also J1.2 (Pin_2)
Other:
- moved on the sheet: R2, R3, R4
Changed lines of the file:
@@
 L Device:R_Small R4
 U 1 1 5EA959CA
-P 5550 2950
-F 0 "R4" V 5354 2950 50  0000 C CNN
-F 1 "10K" V 5445 2950 50  0000 C CNN
-F 2 "" H 5550 2950 50  0001 C CNN
-F 3 "~" H 5550 2950 50  0001 C CNN
-	1    5550 2950
-	0    1    1    0
+P 5200 2750
+F 0 "R4" V 5004 2750 50  0000 C CNN
+F 1 "10K" V 5095 2750 50  0000 C CNN
+F 2 "" H 5200 2750 50  0001 C CNN
+F 3 "~" H 5200 2750 50  0001 C CNN
+	1    5200 2750
+	-1   0    0    1
 $EndComp
 $Comp
 L Device:R_Small R3
 U 1 1 5EA97196
-P 5550 2600
-F 0 "R3" V 5354 2600 50  0000 C CNN
-F 1 "10K" V 5445 2600 50  0000 C CNN
-F 2 "" H 5550 2600 50  0001 C CNN
-F 3 "~" H 5550 2600 50  0001 C CNN
-	1    5550 2600
-	0    1    1    0
+P 5850 2550
+F 0 "R3" V 5654 2550 50  0000 C CNN
+F 1 "10K" V 5745 2550 50  0000 C CNN
+F 2 "" H 5850 2550 50  0001 C CNN
+F 3 "~" H 5850 2550 50  0001 C CNN
+	1    5850 2550
+	-1   0    0    1
 $EndComp
 $Comp
 L Device:R_Small R2
 U 1 1 5EA97679
-P 5550 2250
-F 0 "R2" V 5354 2250 50  0000 C CNN
-F 1 "10K" V 5445 2250 50  0000 C CNN
-F 2 "" H 5550 2250 50  0001 C CNN
-F 3 "~" H 5550 2250 50  0001 C CNN
-	1    5550 2250
-	0    1    1    0
+P 5550 2550
+F 0 "R2" V 5354 2550 50  0000 C CNN
+F 1 "10K" V 5445 2550 50  0000 C CNN
+F 2 "" H 5550 2550 50  0001 C CNN
+F 3 "~" H 5550 2550 50  0001 C CNN
+	1    5550 2550
+	-1   0    0    1
 $EndComp
 $Comp
@@
 Wire Wire Line
 	6050 3250 6050 3150
-Wire Wire Line
-	5750 2950 5650 2950
-Wire Wire Line
-	5450 2950 5200 2950
-Wire Wire Line
-	5200 2950 5200 2550
-Wire Wire Line
-	5200 2550 5100 2550
-Wire Wire Line
-	5450 2600 5300 2600
-Wire Wire Line
-	5300 2600 5300 2450
-Wire Wire Line
-	5300 2450 5100 2450
-Wire Wire Line
-	5450 2250 5300 2250
-Wire Wire Line
-	5300 2250 5300 2350
-Wire Wire Line
-	5300 2350 5100 2350
 $Comp
 L Connector:USB_B_Micro J?
@@
 	6050 2750 6050 2500
 Wire Wire Line
-	5950 2600 5950 2400
-Wire Wire Line
-	5950 2400 6050 2400
-Wire Wire Line
-	5650 2600 5950 2600
-Wire Wire Line
-	5650 2250 5950 2250
-Wire Wire Line
-	5950 2250 5950 2300
-Wire Wire Line
-	5950 2300 6050 2300
-Wire Wire Line
 	6050 2200 6050 1950
 Wire Wire Line
@@
 Wire Wire Line
 	2850 2400 2850 2500
+$Comp
+L power:GND #PWR?
+U 1 1 5EAA0A67
+P 5700 2700
+F 0 "#PWR?" H 5700 2450 50  0001 C CNN
+F 1 "GND" H 5705 2527 50  0000 C CNN
+F 2 "" H 5700 2700 50  0001 C CNN
+F 3 "" H 5700 2700 50  0001 C CNN
+	1    5700 2700
+	1    0    0    -1
+$EndComp
+Wire Wire Line
+	5750 2950 5200 2950
+Wire Wire Line
+	5200 2950 5200 2850
+Wire Wire Line
+	5200 2650 5200 2550
+Wire Wire Line
+	5200 2550 5100 2550
+Wire Wire Line
+	6050 2300 5550 2300
+Wire Wire Line
+	5200 2300 5200 2350
+Wire Wire Line
+	5200 2350 5100 2350
+Wire Wire Line
+	6050 2400 5850 2400
+Wire Wire Line
+	5250 2400 5250 2450
+Wire Wire Line
+	5250 2450 5100 2450
+Wire Wire Line
+	5550 2650 5550 2700
+Wire Wire Line
+	5850 2700 5850 2650
+Wire Wire Line
+	5550 2700 5700 2700
+Connection ~ 5700 2700
+Wire Wire Line
+	5700 2700 5850 2700
+Wire Wire Line
+	5550 2450 5550 2300
+Connection ~ 5550 2300
+Wire Wire Line
+	5550 2300 5200 2300
+Wire Wire Line
+	5850 2450 5850 2400
+Connection ~ 5850 2400
+Wire Wire Line
+	5850 2400 5250 2400
 $EndSCHEMATC
